Commit message: thread pool example

File: launch/mass_spring_box.sdf.xacro (robot description, xacro)
@@ -2,10 +2,10 @@
 <sdf version="1.4" xmlns:xacro="http://www.ros.org/wiki/xacro">
 <model name="mass_spring">
-  <xacro:property name="PI" value="3.1415926535897931"/>
-  <!-- end-effector properties -->
-  <xacro:property name="mass" value="1"/>
-  <xacro:property name="x" value=".1"/>
-  <xacro:property name="y" value=".1"/>
-  <xacro:property name="z" value=".1"/>
+<xacro:property name="PI" value="3.1415926535897931"/>
+<!-- end-effector properties -->
+<xacro:property name="mass" value="1"/>
+<xacro:property name="x" value=".1"/>
+<xacro:property name="y" value=".1"/>
+<xacro:property name="z" value=".1"/>
 <!-- physics parameters -->
 <xacro:arg name="enable_physics_plugin" default="true"/>
@@ -16,5 +16,5 @@
 <xacro:arg name="length" default="1"/>
 <!-- Model plugin for physics -->
-  <xacro:if value="$(arg enable_physics_plugin)">
+<xacro:if value="$(arg enable_physics_plugin)">
     <plugin name="soft_body_physics_plugin" filename="libsoft_body_physics_plugin.so">
         <fxy>$(arg fxy)</fxy>
@@ -25,5 +25,5 @@
         <attach_point>0 0 0</attach_point>
     </plugin>
-  </xacro:if>
+</xacro:if>
     <link name="base_link"/>
     <link name="ee">
